Commit message: more changes to have a urdf compatible to the feetech_ros2_driver

File: ros2_waveshare_bridge/urdf/so-arm101.sample.urdf (robot description, URDF)
Before this commit: robot so_101_arm, 7 links, 6 joints
Joints:
- joint elbow_flex: axis 0 1 0 -> 0 -1 0
- joint wrist_flex: axis 0 1 0 -> 0 -1 0

Commit message: more changes

File: ros2_waveshare_bridge/urdf/so-arm101.sample.urdf (robot description, URDF)
Before this commit: robot so_101_arm, 7 links, 6 joints
Joints:
- joint wrist_roll: axis 1 0 0 -> -1 0 0

Commit message: alignment between approaches

File: ros2_waveshare_bridge/urdf/so-arm101.sample.urdf (robot description, URDF)
Before this commit: robot so_101_arm, 7 links, 6 joints
Joints:
- joint elbow_flex: axis 0 -1 0 -> 0 1 0
- joint shoulder_lift: axis 0 1 0 -> 0 -1 0
- joint wrist_flex: axis 0 -1 0 -> 0 1 0
